Commit message: sixdofarm.urdf

File: sixdofarm/urdf/sixdofarm.urdf (robot description, URDF)
Before this commit: robot sixdofarm, 8 links, 7 joints
Links:
- added link world
- link link4: geometry collision box size=0.05 0.1 0.05; visual box size=0.05 0.1 0.05
Joints:
- added joint world2base: type fixed, parent world, child base
